Commit message: three hokuyo test

File: urdf/three_hokuyo.urdf (robot description, URDF)
Before this commit: robot cartographer_backpack_2d, 5 links, 2 joints
Joints:
- added joint vertical_left_laser_link_joint: type fixed, parent base_link, child vertical_left_laser_link, origin xyz=0.1 -0.2 0.3 rpy=0 1.570796 0 
- added joint vertical_right_laser_link_joint: type fixed, parent base_link, child vertical_right_laser_link, origin xyz=0.1 0.2 0.5 rpy=-1.570796 1.570796 0
- joint horizontal_laser_link_joint: child vertical_left_laser_link -> horizontal_laser_link; origin xyz=0.1 -0.2 0.3 rpy=1.570796 0 -1.570796 -> xyz=0 0 0.75 rpy=0 0 0
