Commit message: velodyne 3d slam
launch, urdf,lua

File: urdf/three_hokuyo_ydy2.urdf (robot description, URDF)
Before this commit: robot cartographer_backpack_2d, 4 links, 3 joints
Links:
- removed link vertical_laser_link
- added link vertical_left_laser_link; visual cylinder length=0.05 radius=0.03
- added link vertical_right_laser_link; visual cylinder length=0.05 radius=0.03
Joints:
- removed joint vertical_laser_link_joint
- added joint vertical_left_laser_link_joint: type fixed, parent base_link, child vertical_left_laser_link, origin xyz=0.1309601  0.2834585  0.3186169 rpy=0.1315    -1.5430    -2.4868
- added joint vertical_right_laser_link_joint: type fixed, parent base_link, child vertical_right_laser_link, origin xyz=0.1446951   0.077  0.5380209 rpy=-0.7076   1.4941    -1.1402
- joint horizontal_laser_link_joint: origin xyz=0.1007 0 0.0558 -> xyz=0.1006602  0.1539847  0. rpy=0.   0.   0.
- joint imu_link_joint: origin xyz=0 0 0 rpy=0 0 0 -> xyz=0 0 0

File: urdf/whubackpack_3d.urdf (robot description, URDF)
Before this commit: robot cartographer_backpack_2d, 4 links, 3 joints
Links:
- removed link horizontal_laser_link
- removed link vertical_laser_link
- added link velodyne_32E_link; visual cylinder length=0.07 radius=0.05
Joints:
- removed joint horizontal_laser_link_joint
- removed joint vertical_laser_link_joint
- added joint velodyne_32E_link_joint: type fixed, parent base_link, child velodyne_32E_link, origin xyz=0. 0. 0.1 rpy=0. 0. 0.0
